File: KiCad/Li-Ion-BatteryPack.sch (KiCad schematic (older format))
At the start: 17 parts, among them J1 Charger, J2 Load, J3 Parallel, J4 BMS Sensor

Commit message: Updates on gerber files.
Other:
- note added: "Charge"
- note added: "Power"
- note removed: "Concentric"
- note removed: "Splitter"
Changed lines of the file:
@@
 Text Notes 3950 5100 0    50   ~ 0
 CL+
-Text Notes 5700 4500 0    50   ~ 0
-Concentric
-Text Notes 5800 4600 0    50   ~ 0
-Splitter
+Text Notes 6050 4500 0    50   ~ 0
+Charge
+Text Notes 6050 4600 0    50   ~ 0
+Power
 Wire Wire Line
 	5550 4600 6300 4600
